File: Coil_speedifier.kicad_pcb (KiCad board)
At the start: 2 copper layers, 149.9 x 87.6 mm, 33 parts, among them J1 Screw_Terminal_01x02, J2 Conn_Coaxial, J3 Screw_Terminal_01x02, Q1 Q_NPN_Darlington_BCE, Q2 Q_NMOS_GDS, Q3 Q_NMOS_GDS, U1 LTV-817, U2 PDS1-S15-S15-M

Commit message: updated to version 8
Other:
- net class Default removed
